Commit message: Added gazebo support for IRB 2400. Added ROS control packages,but PID controllers need tuning

File: abb_irb120_gazebo/urdf/irb120.xacro (robot description, xacro)
@@ -2,11 +2,9 @@
 <robot name="abb_irb120" xmlns:xacro="http://ros.org/wiki/xacro">
 	<xacro:property name="pi" value="3.1415926535897931" />
-	<xacro:include filename="$(find abb_irb120_support)/urdf/irb120_macro.xacro"/>
-	<xacro:include filename="$(find abb_irb120_gazebo)/urdf/abb_irb120.gazebo" />
+	<xacro:include filename="$(find abb_irb120_gazebo)/urdf/irb120_macro.xacro"/>
+	<xacro:include filename="$(find abb_irb120_gazebo)/urdf/irb120.gazebo" />
 	<xacro:include filename="$(find abb_irb120_gazebo)/urdf/materials.xacro" />
-	<xacro:include filename="$(find abb_irb120_gazebo)/urdf/abb_irb120_inertia.xacro"/>
-	<xacro:include filename="$(find abb_irb120_gazebo)/urdf/abb_irb120_transmission.xacro"/>
+	<xacro:include filename="$(find abb_irb120_gazebo)/urdf/irb120_transmission.xacro"/>
 	<xacro:abb_irb120 prefix=""/>
-	<xacro:abb_irb120_inertia prefix=""/>
 	<xacro:abb_irb120_transmission prefix=""/>
 	<!-- Used for fixing robot to Gazebo world -->

File: abb_irb120_gazebo/urdf/irb120_macro.xacro (robot description, xacro)
@@ -14,11 +14,11 @@
 				<origin xyz="0 0 0" rpy="0 0 0"/>
 				<geometry>
-					<mesh filename="package://abb_irb120_support/meshes/irb120/visual/base_link.STL"/>
-				</geometry>
-				<material name="orange"/>
-			</visual>
-			<collision>
-				<geometry>
-					<mesh filename="package://abb_irb120_support/meshes/irb120/collision/base_link.STL"/>
+					<mesh filename="package://abb_irb120_support/meshes/irb120/visual/base_link.stl"/>
+				</geometry>
+				<material name="orange"/>
+			</visual>
+			<collision>
+				<geometry>
+					<mesh filename="package://abb_irb120_support/meshes/irb120/collision/base_link.stl"/>
 				</geometry>
 			</collision>
@@ -35,12 +35,12 @@
 				<origin xyz="0 0 0" rpy="0 0 0"/>
 				<geometry>
-					<mesh filename="package://abb_irb120_support/meshes/irb120/visual/link_1.STL"/>
-				</geometry>
-				<material name="orange"/>
-			</visual>
-			<collision>
-				<origin xyz="0 0 0" rpy="0 0 0"/>
-				<geometry>
-					<mesh filename="package://abb_irb120_support/meshes/irb120/collision/link_1.STL"/>
+					<mesh filename="package://abb_irb120_support/meshes/irb120/visual/link_1.stl"/>
+				</geometry>
+				<material name="orange"/>
+			</visual>
+			<collision>
+				<origin xyz="0 0 0" rpy="0 0 0"/>
+				<geometry>
+					<mesh filename="package://abb_irb120_support/meshes/irb120/collision/link_1.stl"/>
 				</geometry>
 			</collision>
@@ -57,12 +57,12 @@
 				<origin xyz="0 0 0" rpy="0 0 0"/>
 				<geometry>
-					<mesh filename="package://abb_irb120_support/meshes/irb120/visual/link_2.STL"/>
-				</geometry>
-				<material name="orange"/>
-			</visual>
-			<collision>
-				<origin xyz="0 0 0" rpy="0 0 0"/>
-				<geometry>
-					<mesh filename="package://abb_irb120_support/meshes/irb120/collision/link_2.STL"/>
+					<mesh filename="package://abb_irb120_support/meshes/irb120/visual/link_2.stl"/>
+				</geometry>
+				<material name="orange"/>
+			</visual>
+			<collision>
+				<origin xyz="0 0 0" rpy="0 0 0"/>
+				<geometry>
+					<mesh filename="package://abb_irb120_support/meshes/irb120/collision/link_2.stl"/>
 				</geometry>
 			</collision>
@@ -79,12 +79,12 @@
 				<origin xyz="0 0 0" rpy="0 0 0"/>
 				<geometry>
-					<mesh filename="package://abb_irb120_support/meshes/irb120/visual/link_3.STL"/>
-				</geometry>
-				<material name="orange"/>
-			</visual>
-			<collision>
-				<origin xyz="0 0 0" rpy="0 0 0"/>
-				<geometry>
-					<mesh filename="package://abb_irb120_support/meshes/irb120/collision/link_3.STL"/>
+					<mesh filename="package://abb_irb120_support/meshes/irb120/visual/link_3.stl"/>
+				</geometry>
+				<material name="orange"/>
+			</visual>
+			<collision>
+				<origin xyz="0 0 0" rpy="0 0 0"/>
+				<geometry>
+					<mesh filename="package://abb_irb120_support/meshes/irb120/collision/link_3.stl"/>
 				</geometry>
 			</collision>
@@ -101,12 +101,12 @@
 				<origin xyz="0 0 0" rpy="0 0 0"/>
 				<geometry>
-					<mesh filename="package://abb_irb120_support/meshes/irb120/visual/link_4.STL"/>
-				</geometry>
-				<material name="orange"/>
-			</visual>
-			<collision>
-				<origin xyz="0 0 0" rpy="0 0 0"/>
-				<geometry>
-					<mesh filename="package://abb_irb120_support/meshes/irb120/collision/link_4.STL"/>
+					<mesh filename="package://abb_irb120_support/meshes/irb120/visual/link_4.stl"/>
+				</geometry>
+				<material name="orange"/>
+			</visual>
+			<collision>
+				<origin xyz="0 0 0" rpy="0 0 0"/>
+				<geometry>
+					<mesh filename="package://abb_irb120_support/meshes/irb120/collision/link_4.stl"/>
 				</geometry>
 			</collision>
@@ -123,12 +123,12 @@
 				<origin xyz="0 0 0" rpy="0 0 0"/>
 				<geometry>
-					<mesh filename="package://abb_irb120_support/meshes/irb120/visual/link_5.STL"/>
-				</geometry>
-				<material name="orange"/>
-			</visual>
-			<collision>
-				<origin xyz="0 0 0" rpy="0 0 0"/>
-				<geometry>
-					<mesh filename="package://abb_irb120_support/meshes/irb120/collision/link_5.STL"/>
+					<mesh filename="package://abb_irb120_support/meshes/irb120/visual/link_5.stl"/>
+				</geometry>
+				<material name="orange"/>
+			</visual>
+			<collision>
+				<origin xyz="0 0 0" rpy="0 0 0"/>
+				<geometry>
+					<mesh filename="package://abb_irb120_support/meshes/irb120/collision/link_5.stl"/>
 				</geometry>
 			</collision>
@@ -145,5 +145,5 @@
 				<origin xyz="0 0 0" rpy="0 0 0"/>
 				<geometry>
-					<mesh filename="package://abb_irb120_support/meshes/irb120/visual/link_6.STL"/>
+					<mesh filename="package://abb_irb120_support/meshes/irb120/visual/link_6.stl"/>
 				</geometry>
 				<material name="black">
@@ -154,5 +154,5 @@
 				<origin xyz="0 0 0" rpy="0 0 0"/>
 				<geometry>
-					<mesh filename="package://abb_irb120_support/meshes/irb120/collision/link_6.STL"/>
+					<mesh filename="package://abb_irb120_support/meshes/irb120/collision/link_6.stl"/>
 				</geometry>
 			</collision>
